Commit message: Completed Task A

File: nuturtle_description/urdf/diff_drive.urdf.xacro (robot description, xacro)
@@ -7,55 +7,62 @@
 <!-- name dimension['wheel_radius'] to radius for simplicity -->
 <xacro:property name="radius" value="${dimension['wheel_radius']}" />
-<!-- prism link -->
-<link name="prism">
+<!-- The actual width of the base -->
+<xacro:property name="base_width" value="${dimension['wheel_base'] - dimension['wheel_width']}" />
+<!-- Define caster 'radius' - the length of the cylinder -->
+<xacro:property name="caster_radius" value="${radius - dimension['chassis_thickness']/2}" />
+<!-- base_link -->
+<link name="base_link">
     <inertial>
-        <mass value="6"/>
-        <origin rpy="0 0 0" xyz="0 0 0"/>
-        <inertia ixx="${6*(dimension['wheel_base']**2+dimension['chassis_thickness']**2)/12}" ixy="0" ixz="0"
-            iyy="${6*(dimension['chassis_length']**2+dimension['chassis_thickness']**2)/12}" iyz="0" izz="${6*(dimension['chassis_length']**2+dimension['wheel_base']**2)/12}"/>
+        <mass value="1"/>
+        <origin rpy="0 0 0" xyz="${(dimension['chassis_length']/2 - radius)} 0 0"/>
+        <inertia ixx="${1*(base_width**2+dimension['chassis_thickness']**2)/12}" ixy="0" ixz="0"
+            iyy="${1*(dimension['chassis_length']**2+dimension['chassis_thickness']**2)/12}" iyz="0" izz="${1*(dimension['chassis_length']**2+base_width**2)/12}"/>
     </inertial>
-    <collision name="prism_collision">
+    <collision name="base_link_collision">
+        <origin rpy="0 0 0" xyz="${(dimension['chassis_length']/2 - radius)} 0 0" />
         <geometry>
-            <box size="${dimension['chassis_length']} ${dimension['wheel_base']} ${dimension['chassis_thickness']}"/>
+            <box size="${dimension['chassis_length']} ${base_width} ${dimension['chassis_thickness']}"/>
         </geometry>
     </collision>
-    <visual name="prism_visual">
-        <origin rpy="0 0 0" xyz="0 0 0"/>
+    <visual name="base_link_visual">
+        <!-- Learned: orgin here is displaced from the orgin of the last joint frame -->
+        <origin rpy="0 0 0" xyz="${(dimension['chassis_length']/2 - radius)} 0 0"/>
         <geometry>
-            <box size="${dimension['chassis_length']} ${dimension['wheel_base']} ${dimension['chassis_thickness']}"/>
+            <box size="${dimension['chassis_length']} ${base_width} ${dimension['chassis_thickness']}"/>
         </geometry>
-        <material name="green">
-                <color rgba="0 1 0 1" />
+        <material name="blue">
+                <color rgba="0 0 1 1" />
         </material>
     </visual>
 </link>
 <!-- caster 1 joint and link -->
-<joint name="prism_caster1" type="fixed">
-    <origin xyz="-0.2 0 ${-(dimension['chassis_thickness']/2+0.025)}" rpy="0 0 0" />
-    <parent link="prism" />
+<joint name="base_link_caster1" type="fixed">
+    <!-- Learned: it is displaced from the last joint frame -->
+    <origin xyz="${dimension['chassis_length'] - radius - caster_radius} 0 ${-(dimension['chassis_thickness']/2+caster_radius/2)}" rpy="0 0 0" />
+    <parent link="base_link" />
     <child link="caster1" />
 </joint>
 <xacro:link_caster name="caster1" />
 <!-- caster 2 joint and link -->
-<joint name="prism_caster2" type="fixed">
-    <origin xyz="-0.2 0 ${dimension['chassis_thickness']/2+0.025}" rpy="0 0 0" />
-    <parent link="prism" />
+<joint name="base_link_caster2" type="fixed">
+    <origin xyz="${dimension['chassis_length'] - radius - caster_radius} 0 ${dimension['chassis_thickness']/2+caster_radius/2}" rpy="0 0 0" />
+    <parent link="base_link" />
     <child link="caster2" />
 </joint>
 <xacro:link_caster name="caster2" />
 <!-- left wheel joint and link -->
-<joint name="prism_right_wheel" type="continuous">
-    <origin rpy="${pi/2} 0 0" xyz="0.1 ${-(dimension['wheel_base']/2+0.02)} 0"/>
-    <parent link="prism"/>
+<joint name="right_wheel_axle" type="continuous">
+    <origin rpy="0 0 0" xyz="0 ${-(dimension['wheel_base']/2)} 0"/>
+    <parent link="base_link"/>
     <child link="right_wheel" />
-    <axis rpy="0 0 0" xyz="0 0 -1"/>
+    <axis rpy="0 0 0" xyz="0 1 0"/>
 </joint>
 <xacro:link_wheel name="right_wheel" />
 <!-- right wheel joint and link -->
-<joint name="prism_left_wheel" type="continuous">
-    <origin rpy="${-pi/2} 0 0" xyz="0.1 ${dimension['wheel_base']/2+0.02} 0"/>
-    <parent link="prism"/>
+<joint name="left_wheel_axle" type="continuous">
+    <origin rpy="0 0 0" xyz="0 ${dimension['wheel_base']/2} 0"/>
+    <parent link="base_link"/>
     <child link="left_wheel" />
-    <axis rpy="0 0 0" xyz="0 0 1"/>
+    <axis rpy="0 0 0" xyz="0 1 0"/>
 </joint>
 <xacro:link_wheel name="left_wheel" />

File: nuturtle_description/urdf/diff_drive_macro.xacro (robot description, xacro)
@@ -6,17 +6,17 @@
             <inertial>
                 <mass value="0.2"/>
-                <origin rpy="0 0 0" xyz="0 0 0"/>
-                <inertia ixx="${0.2*(3*radius**2+0.04**2)/12}" ixy="0" ixz="0" iyy="${0.2*(3*radius**2+0.04**2)/12}" iyz="0" izz="${0.2*radius**2/2}"/>
+                <origin rpy="${-pi/2} 0 0" xyz="0 0 0"/>
+                <inertia ixx="${0.2*(3*radius**2+dimension['wheel_width']**2)/12}" ixy="0" ixz="0" iyy="${0.2*(3*radius**2+dimension['wheel_width']**2)/12}" iyz="0" izz="${0.2*radius**2/2}"/>
             </inertial>
             <collision name="${name}_collision">
-                <origin rpy="0 0 0" xyz="0 0 0" />
+                <origin rpy="${-pi/2} 0 0" xyz="0 0 0" />
                 <geometry>
-                    <cylinder length="0.04" radius="${radius}"/>
+                    <cylinder length="${dimension['wheel_width']}" radius="${radius}"/>
                 </geometry>
             </collision>
             <visual name="${name}_visual">
-                <origin rpy="0 0 0" xyz="0 0 0"/>
+                <origin rpy="${-pi/2} 0 0" xyz="0 0 0"/>
                 <geometry>
-                    <cylinder length="0.04" radius="${radius}"/>
+                    <cylinder length="${dimension['wheel_width']}" radius="${radius}"/>
                 </geometry>
                 <material name="red">
@@ -32,10 +32,10 @@
                 <mass value="0.1"/>
                 <origin rpy="0 0 0" xyz="0 0 0"/>
-                <inertia ixx="${0.1*(3*0.05**2+0.05**2)/12}" ixy="0" ixz="0" iyy="${0.1*(3*0.05**2+0.05**2)/12}" iyz="0" izz="${0.1*0.05**2/2}"/>
+                <inertia ixx="${0.1*(3*caster_radius**2+caster_radius**2)/12}" ixy="0" ixz="0" iyy="${0.1*(3*caster_radius**2+caster_radius**2)/12}" iyz="0" izz="${0.1*caster_radius**2/2}"/>
             </inertial>
             <collision name="${name}_collision">
                 <origin rpy="0 0 0" xyz="0 0 0" />
                 <geometry>
-                    <cylinder length="0.05" radius="0.05"/>
+                    <cylinder length="${caster_radius}" radius="${caster_radius}"/>
                 </geometry>
             </collision>
@@ -43,8 +43,8 @@
                 <origin rpy="0 0 0" xyz="0 0 0"/>
                 <geometry>
-                    <cylinder length="0.05" radius="0.05"/>
+                    <cylinder length="${caster_radius}" radius="${caster_radius}"/>
                 </geometry>
-                <material name="red">
-                        <color rgba="1 0 0 1" />
+                <material name="green">
+                        <color rgba="0 1 0 1" />
                 </material>
             </visual>

Commit message: added dummy link

File: nuturtle_description/urdf/diff_drive.urdf.xacro (robot description, xacro)
@@ -11,4 +11,11 @@
 <!-- Define caster 'radius' - the length of the cylinder -->
 <xacro:property name="caster_radius" value="${radius - dimension['chassis_thickness']/2}" />
+<!-- add a dummy link for KDL -->
+<link name="dummy">
+</link>
+<joint name="dummy_joint" type="fixed">
+    <parent link="dummy"/>
+    <child link="base_link"/>
+</joint>
 <!-- base_link -->
 <link name="base_link">

Commit message: Modified urdf

File: nuturtle_description/urdf/diff_drive.urdf.xacro (robot description, xacro)
@@ -10,14 +10,23 @@
 <xacro:property name="base_width" value="${dimension['wheel_base'] - dimension['wheel_width']}" />
 <!-- Define caster 'radius' - the length of the cylinder -->
-<xacro:property name="caster_radius" value="${radius - dimension['chassis_thickness']/2}" />
-<!-- add a dummy link for KDL -->
-<link name="dummy">
+<xacro:property name="caster_radius" value="${radius - dimension['wheel_axle_offset']}" />
+<!-- add a inertial-less base link for KDL -->
+<link name="base_link">
 </link>
-<joint name="dummy_joint" type="fixed">
-    <parent link="dummy"/>
-    <child link="base_link"/>
+<joint name="base_link_base_link_dummy_joint" type="fixed">
+    <origin xyz="${-(dimension['chassis_length']/2 - radius)} 0 ${radius - dimension['wheel_axle_offset'] + dimension['chassis_thickness']/2}" rpy="0 0 0" />
+    <parent link="base_link"/>
+    <child link="base_link_dummy"/>
 </joint>
-<!-- base_link -->
-<link name="base_link">
+<!-- add a base scan link -->
+<joint name="base_link_base_scan_joint" type="fixed">
+    <origin xyz="0 0 ${radius - dimension['wheel_axle_offset'] + dimension['chassis_thickness']}" rpy="0 0 0" />
+    <parent link="base_link"/>
+    <child link="base_scan"/>
+</joint>
+<link name="base_scan">
+</link>
+<!-- base_link_dummy -->
+<link name="base_link_dummy">
     <inertial>
         <mass value="1"/>
@@ -26,5 +35,5 @@
             iyy="${1*(dimension['chassis_length']**2+dimension['chassis_thickness']**2)/12}" iyz="0" izz="${1*(dimension['chassis_length']**2+base_width**2)/12}"/>
     </inertial>
-    <collision name="base_link_collision">
+    <collision name="base_link_dummy_collision">
         <origin rpy="0 0 0" xyz="${(dimension['chassis_length']/2 - radius)} 0 0" />
         <geometry>
@@ -32,5 +41,5 @@
         </geometry>
     </collision>
-    <visual name="base_link_visual">
+    <visual name="base_link_dummy_visual">
         <!-- Learned: orgin here is displaced from the orgin of the last joint frame -->
         <origin rpy="0 0 0" xyz="${(dimension['chassis_length']/2 - radius)} 0 0"/>
@@ -44,15 +53,15 @@
 </link>
 <!-- caster 1 joint and link -->
-<joint name="base_link_caster1" type="fixed">
+<joint name="base_link_dummy_caster1" type="fixed">
     <!-- Learned: it is displaced from the last joint frame -->
     <origin xyz="${dimension['chassis_length'] - radius - caster_radius} 0 ${-(dimension['chassis_thickness']/2+caster_radius/2)}" rpy="0 0 0" />
-    <parent link="base_link" />
+    <parent link="base_link_dummy" />
     <child link="caster1" />
 </joint>
 <xacro:link_caster name="caster1" />
 <!-- caster 2 joint and link -->
-<joint name="base_link_caster2" type="fixed">
+<joint name="base_link_dummy_caster2" type="fixed">
     <origin xyz="${dimension['chassis_length'] - radius - caster_radius} 0 ${dimension['chassis_thickness']/2+caster_radius/2}" rpy="0 0 0" />
-    <parent link="base_link" />
+    <parent link="base_link_dummy" />
     <child link="caster2" />
 </joint>
@@ -60,6 +69,6 @@
 <!-- left wheel joint and link -->
 <joint name="right_wheel_axle" type="continuous">
-    <origin rpy="0 0 0" xyz="0 ${-(dimension['wheel_base']/2)} 0"/>
-    <parent link="base_link"/>
+    <origin rpy="0 0 0" xyz="0 ${-(dimension['wheel_base']/2)} ${-(dimension['chassis_thickness']/2) + dimension['wheel_axle_offset']}"/>
+    <parent link="base_link_dummy"/>
     <child link="right_wheel" />
     <axis rpy="0 0 0" xyz="0 1 0"/>
@@ -68,6 +77,6 @@
 <!-- right wheel joint and link -->
 <joint name="left_wheel_axle" type="continuous">
-    <origin rpy="0 0 0" xyz="0 ${dimension['wheel_base']/2} 0"/>
-    <parent link="base_link"/>
+    <origin rpy="0 0 0" xyz="0 ${dimension['wheel_base']/2} ${-(dimension['chassis_thickness']/2) + dimension['wheel_axle_offset']}"/>
+    <parent link="base_link_dummy"/>
     <child link="left_wheel" />
     <axis rpy="0 0 0" xyz="0 1 0"/>

Commit message: added nuturtle_gazebo

File: nuturtle_description/urdf/diff_drive.urdf.xacro (robot description, xacro)
@@ -57,5 +57,5 @@
 <joint name="base_link_dummy_caster1" type="fixed">
     <!-- Learned: it is displaced from the last joint frame -->
-    <origin xyz="${dimension['chassis_length'] - radius - caster_radius} 0 ${-(dimension['chassis_thickness']/2+caster_radius/2)}" rpy="0 0 0" />
+    <origin xyz="${dimension['chassis_length'] - radius - caster_radius} 0 ${-(dimension['chassis_thickness']/2)}" rpy="0 0 0" />
     <parent link="base_link_dummy" />
     <child link="caster1" />
@@ -64,5 +64,5 @@
 <!-- caster 2 joint and link -->
 <joint name="base_link_dummy_caster2" type="fixed">
-    <origin xyz="${dimension['chassis_length'] - radius - caster_radius} 0 ${dimension['chassis_thickness']/2+caster_radius/2}" rpy="0 0 0" />
+    <origin xyz="${dimension['chassis_length'] - radius - caster_radius} 0 ${dimension['chassis_thickness']/2}" rpy="0 0 0" />
     <parent link="base_link_dummy" />
     <child link="caster2" />

File: nuturtle_description/urdf/diff_drive_macro.xacro (robot description, xacro)
@@ -32,10 +32,10 @@
                 <mass value="0.1"/>
                 <origin rpy="0 0 0" xyz="0 0 0"/>
-                <inertia ixx="${0.1*(3*caster_radius**2+caster_radius**2)/12}" ixy="0" ixz="0" iyy="${0.1*(3*caster_radius**2+caster_radius**2)/12}" iyz="0" izz="${0.1*caster_radius**2/2}"/>
+                <inertia ixx="${(2.0/5.0)*0.1*caster_radius**2}" ixy="0" ixz="0" iyy="${(2.0/5.0)*0.1*caster_radius**2}" iyz="0" izz="${(2.0/5.0)*0.1*caster_radius**2}"/>
             </inertial>
             <collision name="${name}_collision">
                 <origin rpy="0 0 0" xyz="0 0 0" />
                 <geometry>
-                    <cylinder length="${caster_radius}" radius="${caster_radius}"/>
+                    <sphere radius="${caster_radius}"/>
                 </geometry>
             </collision>
@@ -43,5 +43,5 @@
                 <origin rpy="0 0 0" xyz="0 0 0"/>
                 <geometry>
-                    <cylinder length="${caster_radius}" radius="${caster_radius}"/>
+                    <sphere radius="${caster_radius}"/>
                 </geometry>
                 <material name="green">

Commit message: completed clustering

File: nuturtle_description/urdf/diff_drive.urdf.xacro (robot description, xacro)
@@ -28,4 +28,9 @@
 </joint>
 <link name="base_scan">
+    <visual name="base_scan_visual">
+        <geometry>
+            <cylinder radius="0.01" length="0.01"/>
+        </geometry>
+    </visual>
 </link>
 <!-- base_link_dummy -->
